File: kicad/IOs.sch (KiCad schematic (older format))
At the start: 57 parts, among them J1 Screw_Terminal_01x04, J2 Screw_Terminal_01x04, J3 Screw_Terminal_01x04, J4 Screw_Terminal_01x04, J5 Screw_Terminal_01x04, J6 Screw_Terminal_01x04, Q1 BSS306NH, Q2 BSS306NH, Q3 BSS306NH, Q4 BSS306NH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

Commit message: Added pullups for I2C
Parts:
- U1, U2, U3: footprint Package_SO:SOIC-8-1EP_3.9x4.9mm_P1.27mm_EP2.29x3mm -> mosfet_drivers:IX4340NE
Changed lines of the file:
@@
 F 0 "U1" H 5200 4965 50  0000 C CNN
 F 1 "IX4340NE" H 5200 4874 50  0000 C CNN
-F 2 "Package_SO:SOIC-8-1EP_3.9x4.9mm_P1.27mm_EP2.29x3mm" H 5150 4600 50  0001 C CNN
+F 2 "mosfet_drivers:IX4340NE" H 5150 4600 50  0001 C CNN
 F 3 "" H 5150 4600 50  0001 C CNN
 	1    5200 4600
@@
 F 0 "U3" H 8200 4965 50  0000 C CNN
 F 1 "IX4340NE" H 8200 4874 50  0000 C CNN
-F 2 "Package_SO:SOIC-8-1EP_3.9x4.9mm_P1.27mm_EP2.29x3mm" H 8150 4600 50  0001 C CNN
+F 2 "mosfet_drivers:IX4340NE" H 8150 4600 50  0001 C CNN
 F 3 "" H 8150 4600 50  0001 C CNN
 	1    8200 4600
@@
 F 0 "U2" H 5200 6965 50  0000 C CNN
 F 1 "IX4340NE" H 5200 6874 50  0000 C CNN
-F 2 "Package_SO:SOIC-8-1EP_3.9x4.9mm_P1.27mm_EP2.29x3mm" H 5150 6600 50  0001 C CNN
+F 2 "mosfet_drivers:IX4340NE" H 5150 6600 50  0001 C CNN
 F 3 "" H 5150 6600 50  0001 C CNN
 	1    5200 6600
