File: kicad/mcu.sch (KiCad schematic (older format))
At the start: 3 parts, among them J10 Conn_01x04_Male, SW1 SW_Push, U4 ESP32DevKitCV4

Commit message: Added pullups for I2C
Parts:
- added R28, R29: 3k3, Resistor_SMD:R_0805_2012Metric_Pad1.15x1.40mm_HandSolder, symbol Device:R
Connections:
- net +3V3: now also R28.1, R29.1
- net SCL: now also R29.2
- net SDA: now also R28.2
Changed lines of the file:
@@
 Wire Wire Line
 	5100 3300 5700 3300
-Wire Wire Line
-	6500 4000 6900 4000
-Wire Wire Line
-	6500 3900 6900 3900
 Text Label 6900 4000 0    50   ~ 0
 SCL
@@
 Wire Wire Line
 	5600 3200 5400 3200
+Wire Wire Line
+	6500 3900 7350 3900
+$Comp
+L Device:R R28
+U 1 1 61E5E901
+P 7350 3750
+F 0 "R28" H 7420 3796 50  0000 L CNN
+F 1 "3k3" H 7420 3705 50  0000 L CNN
+F 2 "Resistor_SMD:R_0805_2012Metric_Pad1.15x1.40mm_HandSolder" V 7280 3750 50  0001 C CNN
+F 3 "~" H 7350 3750 50  0001 C CNN
+	1    7350 3750
+	1    0    0    -1
+$EndComp
+$Comp
+L Device:R R29
+U 1 1 61E5F0E3
+P 7575 3850
+F 0 "R29" H 7645 3896 50  0000 L CNN
+F 1 "3k3" H 7645 3805 50  0000 L CNN
+F 2 "Resistor_SMD:R_0805_2012Metric_Pad1.15x1.40mm_HandSolder" V 7505 3850 50  0001 C CNN
+F 3 "~" H 7575 3850 50  0001 C CNN
+	1    7575 3850
+	1    0    0    -1
+$EndComp
+Wire Wire Line
+	6500 4000 7575 4000
+Wire Wire Line
+	7575 3700 7575 3575
+Wire Wire Line
+	7350 3600 7350 3575
+Wire Wire Line
+	7350 3575 7575 3575
+Text Label 7450 3575 0    50   ~ 0
+3V3
 $EndSCHEMATC
